File: hardware/logicboard/gb-001.brd (EAGLE design)
At the start: 92 x 58 mm, 8 parts

Commit message: Added capacitors.
Parts:
- added C1, C2: (no value), rcl:C025-025X050
- R1, R2: value (none) -> 1k
Connections:
- net GND: now also C1.2, C2.2
- net VCC: now also C1.1
- net VCC/2: now also C2.1
Routing:
- net GND: track 154.4 -> 167.3 mm
- net GB04: track 43.2 -> 53.0 mm
- net GB00: track 55.6 -> 45.9 mm
- net VCC: track 11.7 -> 21.3 mm
- net GB09: track 63.7 -> 54.4 mm
- net VCC/2: track 24.3 -> 30.5 mm
- net GB07: track 39.7 -> 44.8 mm
- net GB14: track 44.0 -> 39.4 mm
- net GB05: track 41.5 -> 37.4 mm
- net GB06: track 37.6 -> 41.3 mm
- net VCC2LED: track 28.9 -> 25.5 mm
- net GB12: track 42.1 -> 44.5 mm
- net GB11: track 60.2 -> 61.3 mm
- net GB08: track 46.0 -> 46.9 mm
- net GB10: track 56.4 -> 57.1 mm
